File: Lawo 28x13.sch (KiCad schematic (older format))
At the start: 18 parts, among them IC1 FP2800a, J1 Solder_Jumper, J2 Solder_Jumper, J3 Solder_Jumper, J4 Solder_Jumper, J5 Solder_Jumper, J6 Solder_Jumper, U1 TSR-1

Commit message: Updated schematic for upgraded KiCad version and rework of many traces and pin assignments
- KiCad version upgrade
 - EESchema Schematic File Version 4
 - KiCad 5.0.0-rc3-dev
 - symbols and footprint exchanged to newer versions
- board changes
 - changed pin assignments for the set pins (swapped group of FP2800a 2a-g and 3a-g)
 - additional enable pins E_zR and E_yZ for spare connections
 - additional traces for one more set and one reset pin, routing to I1 selectable via solder jumper
 - increased trace widths
 - increased board size
 - silkscreen updates (outlines, component values, pin labels, ...)
 - bunch of vias added to shorten ground loops
- updated plots of the upgraded schematic, including images of the 3D viewer
Parts:
- added I3: Spare Enable, Socket_Strips:Socket_Strip_Straight_1x02_Pitch2.54mm, symbol Connector:Conn_01x02
- C1: value 0.22uF -> 0.22μF
- C2: value 22uF -> 22μF
Connections:
- net labels added: COL_ENABLE_yR, COL_ENABLE_zR
- wire segments 168 -> 172
- no-connect marks 3 -> 1
Changed lines of the file:
@@
 Title "Lawo 28x13 Flip Dot Interface"
 Date "2019-01-21"
-Rev "0.12"
+Rev "1.1.0"
 Comp "Flip-The-Dot"
 Comment1 "Robert Römer"
@@
 $EndComp
 NoConn ~ 7200 1400
-NoConn ~ 3300 1800
-NoConn ~ 2800 1900
 $Comp
 L power:GND #PWR01
@@
 P 8200 5550
 F 0 "C2" H 8210 5620 50  0000 L CNN
-F 1 "22uF" V 8400 5450 50  0000 L CNN
+F 1 "22μF" V 8400 5450 50  0000 L CNN
 F 2 "Capacitors_THT:CP_Radial_D5.0mm_P2.50mm" H 8200 5550 60  0001 C CNN
 F 3 "" H 8200 5550 60  0000 C CNN
@@
 P 9750 3000
 F 0 "C1" H 9775 3100 50  0000 L CNN
-F 1 "0.22uF" H 9775 2900 50  0000 L CNN
+F 1 "0.22μF" H 9775 2900 50  0000 L CNN
 F 2 "Capacitors_THT:C_Disc_D3.4mm_W2.1mm_P2.50mm" H 9788 2850 50  0001 C CNN
 F 3 "" H 9750 3000 50  0000 C CNN
@@
 L power:GND #PWR06
 U 1 1 57D72A87
-P 4000 1600
-F 0 "#PWR06" H 4000 1350 50  0001 C CNN
-F 1 "GND" V 4000 1410 50  0000 C CNN
-F 2 "" H 4000 1600 60  0000 C CNN
-F 3 "" H 4000 1600 60  0000 C CNN
-	1    4000 1600
+P 4100 1600
+F 0 "#PWR06" H 4100 1350 50  0001 C CNN
+F 1 "GND" V 4100 1410 50  0000 C CNN
+F 2 "" H 4100 1600 60  0000 C CNN
+F 3 "" H 4100 1600 60  0000 C CNN
+	1    4100 1600
 	0    -1   1    0
 $EndComp
@@
 	6300 4800 6600 4800
 Wire Wire Line
-	3300 1600 4000 1600
-Wire Wire Line
 	1700 1700 2800 1700
 Wire Wire Line
@@
 Wire Notes Line
 	3300 4800 3300 7200
-Wire Notes Line
-	700  4800 700  7200
-Wire Notes Line
-	700  7200 3000 7200
-Wire Notes Line
-	3000 7200 3000 4800
 Text Notes 3400 5000 0    60   ~ 0
 Power Levels
@@
 	7400 4800 7800 4800
 Connection ~ 7800 4800
+Text GLabel 3600 1800 2    60   Input ~ 0
+COL_ENABLE_zR
+Text GLabel 2500 1900 0    60   Input ~ 0
+COL_ENABLE_yR
+Wire Wire Line
+	2500 1900 2800 1900
+Wire Wire Line
+	3300 1800 3600 1800
+$Comp
+L Connector:Conn_01x02 I3
+U 1 1 5C610766
+P 1300 7350
+F 0 "I3" H 1300 7450 50  0000 C CNN
+F 1 "Spare Enable" V 1400 7350 50  0000 C CNN
+F 2 "Socket_Strips:Socket_Strip_Straight_1x02_Pitch2.54mm" V 1500 7350 60  0001 C CNN
+F 3 "" H 1300 7350 60  0000 C CNN
+	1    1300 7350
+	-1   0    0    -1
+$EndComp
+Text GLabel 1900 7350 2    60   Output ~ 0
+COL_ENABLE_yR
+Text GLabel 1900 7450 2    60   Output ~ 0
+COL_ENABLE_zR
+Wire Wire Line
+	1900 7450 1500 7450
+Wire Wire Line
+	1500 7350 1900 7350
+Wire Notes Line
+	3000 7650 700  7650
+Wire Notes Line
+	700  4800 700  7650
+Wire Notes Line
+	3000 4800 3000 7650
+Wire Wire Line
+	3300 1600 4100 1600
 $EndSCHEMATC
