File: Lawo 28x13 Interface.sch (KiCad schematic (older format))
At the start: 19 parts, among them IC1 FP2800a, J1 Solder_Jumper, J2 Solder_Jumper, J3 Solder_Jumper, J4 Solder_Jumper, J5 Solder_Jumper, J6 Solder_Jumper, U1 TSR-1

Commit message: Renamed enable pins and slightly modified traces and silk screen.
Connections:
- net labels added: COL_ENABLE_A, COL_ENABLE_B, COL_ENABLE_C, COL_ENABLE_D
- net labels removed: COL_ENABLE_mR, COL_ENABLE_oR, COL_ENABLE_yR, COL_ENABLE_zR
Changed lines of the file:
@@
 encoding utf-8
 Sheet 1 1
-Title "Lawo 28x13 Flip Dot Interface"
-Date "2019-04-27"
-Rev "1.1.1"
+Title "Lawo 50pin Flip Dot Interface (FP2800a)"
+Date "2019-06-23"
+Rev "1.1.2"
 Comp "Flip-The-Dot"
 Comment1 "Robert Römer"
-Comment2 "Interface to control a Lawo flip dot matrix with a 28x13 resolution."
+Comment2 "Interface to control Lawo flip dot matrixes with 50pin connectors and up to 28x14 dots each."
 Comment3 ""
 Comment4 ""
@@
 COL_B1
 Text GLabel 2500 1800 0    60   Input ~ 0
-COL_ENABLE_oR
+COL_ENABLE_A
 Text GLabel 1900 5900 2    60   Output ~ 0
 ROW_A1
@@
 $EndComp
 Text GLabel 3600 1900 2    60   Input ~ 0
-COL_ENABLE_mR
+COL_ENABLE_D
 Text GLabel 1900 6500 2    60   Output ~ 0
 COL_DATA
@@
 $EndComp
 Text GLabel 1900 6300 2    60   Output ~ 0
-COL_ENABLE_mR
+COL_ENABLE_A
 Text GLabel 1900 6400 2    60   Output ~ 0
-COL_ENABLE_oR
+COL_ENABLE_D
 $Comp
 L device:R R1
@@
 Connection ~ 7800 4800
 Text GLabel 3600 1800 2    60   Input ~ 0
-COL_ENABLE_zR
+COL_ENABLE_B
 Text GLabel 2500 1900 0    60   Input ~ 0
-COL_ENABLE_yR
+COL_ENABLE_C
 Wire Wire Line
 	2500 1900 2800 1900
@@
 $EndComp
 Text GLabel 1900 7350 2    60   Output ~ 0
-COL_ENABLE_yR
+COL_ENABLE_B
 Text GLabel 1900 7450 2    60   Output ~ 0
-COL_ENABLE_zR
+COL_ENABLE_C
 Wire Wire Line
 	1900 7450 1500 7450
